File: temp_compare_circuit/temp_compare_circuit.sch (KiCad schematic (older format))
At the start: 188 parts

Commit message: Add shift register
Parts:
- added U? (x64): 4081, symbol 4xxx:4081
- added U? (x64): 4070, symbol 4xxx:4070
- added U? (x32): 74LS04, symbol 74xx:74LS04
- gave numbers to parts that had none: 188
Connections:
- new net: U?.1, U?.2 (x32)
- new net: U?.1, U?.3 (x32)
- new net: U?.2, U?.3 (x64)
- new net CLK: U?.1, U?.1, U?.1, U?.1, U?.1, U?.1, U?.1, U?.1, U?.1, U?.1, U?.1, U?.1, U?.1, U?.1, U?.1, U?.1, U?.1, U?.1, U?.1, U?.1, U?.1, U?.1, U?.1, U?.1, U?.1, U?.1, U?.1, U?.1, U?.1, U?.1, U?.1, U?.1, U?.2, U?.2, U?.2, U?.2, U?.2, U?.2, U?.2, U?.2, U?.2, U?.2, U?.2, U?.2, U?.2, U?.2, U?.2, U?.2, U?.2, U?.2, U?.2, U?.2, U?.2, U?.2, U?.2, U?.2, U?.2, U?.2, U?.2, U?.2, U?.2, U?.2, U?.2, U?.2
- new net Signal_In: U?.1, U?.2
- new net Temp[0]: U?.1, U?.1, U?.1, U?.1, U?.1, U?.1, U?.1, U?.1, U?.2, U?.2, U?.2, U?.2, U?.3, U?.3, U?.3, U?.3
- new net Temp[1]: U?.1, U?.1, U?.1, U?.1, U?.1, U?.1, U?.1, U?.1, U?.2, U?.2, U?.2, U?.2, U?.3, U?.3, U?.3, U?.3
- new net Temp[2]: U?.1, U?.1, U?.1, U?.1, U?.1, U?.1, U?.1, U?.1, U?.2, U?.2, U?.2, U?.2, U?.3, U?.3, U?.3, U?.3
- new net Temp[3]: U?.1, U?.1, U?.1, U?.1, U?.1, U?.1, U?.1, U?.1, U?.2, U?.2, U?.2, U?.2, U?.3, U?.3, U?.3, U?.3
- new net Temp[4]: U?.1, U?.1, U?.1, U?.1, U?.1, U?.1, U?.1, U?.1, U?.2, U?.2, U?.2, U?.2, U?.3, U?.3, U?.3, U?.3
- new net Temp[5]: U?.1, U?.1, U?.1, U?.1, U?.1, U?.1, U?.1, U?.1, U?.2, U?.2, U?.2, U?.2, U?.3, U?.3, U?.3, U?.3
- new net Temp[6]: U?.1, U?.1, U?.1, U?.1, U?.1, U?.1, U?.1, U?.1, U?.2, U?.2, U?.2, U?.2, U?.3, U?.3, U?.3, U?.3
- new net Temp[7]: U?.1, U?.1, U?.1, U?.1, U?.1, U?.1, U?.1, U?.2, U?.2, U?.2, U?.3, U?.3, U?.3, U?.3
Other:
- note added: "Shift Register Signal Input"
- note added: "TEMP1"
- note added: "TEMP2"
- note added: "TEMP3"
- note added: "TEMP4"
- moved on the sheet: U100A, U101A, U102A, U103A, U104A, U105A, U106A, U107A, U108A, U109A, U10A, U110A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
